Commit message: MujocoSystem gripper controller fixes

File: aic_assets/models/Robotiq Hand-E/robotiq_hande.ros2_control.xacro (robot description, xacro)
@@ -25,4 +25,14 @@
         </state_interface>
       </joint>
+      <joint name="${tf_prefix}right_finger_joint">
+        <param name="mimic">${tf_prefix}left_finger_joint</param>
+        <param name="multiplier">1</param>
+        <state_interface name="position">
+          <param name="initial_value">${initial_pos}</param>
+        </state_interface>
+        <state_interface name="velocity">
+          <param name="initial_value">0.0</param>
+        </state_interface>
+      </joint>
     </ros2_control>
   </xacro:macro>

File: aic_assets/models/Robotiq Hand-E/robotiq_hande_macro.xacro (robot description, xacro)
@@ -3,4 +3,8 @@
   <xacro:include filename="$(find aic_assets)/models/Robotiq Hand-E/robotiq_hande.ros2_control.xacro"/>
   <xacro:macro name="robotiq_hande" params="name tf_prefix grip_pos_min grip_pos_max grip_vel_max grip_effort_min grip_effort_max initial_pos hardware_plugin:='gz_ros2_control/GazeboSimSystem'">
+    <!-- Conditional effort limits based on hardware_plugin -->
+    <xacro:property name="is_mujoco" value="${hardware_plugin == 'mujoco_ros2_control/MujocoSystem'}"/>
+    <xacro:property name="grip_effort_min" value="${2 if is_mujoco else 20}"/>
+    <xacro:property name="grip_effort_max" value="130"/>
     <xacro:robotiq_hande_ros2_control
       name="${name}"
